File: PR-16PP.sch (KiCad schematic (older format))
At the start: 26 parts, among them J1 THERM, J2 BATTERY, U1 TP4056, U2 DW01A

Commit message: finish basic schematic
Parts:
- added C5, C6: 4.7uF, symbol Device:C_Small
- added C7, C8: 1uF, symbol Device:C_Small
- added C9: 100n, symbol Device:C_Small
- added D1, D? (x15): SM4007PL, symbol Device:D_Small
- added J3: SWD, symbol Connector:Conn_01x03_Male
- added MX1, MX? (x15): MX-NoLED, symbol MX_Alps_Hybrid:MX-NoLED
- added R10: 806k, symbol Device:R_Small
- added R11: 2M, symbol Device:R_Small
- added SW1: RESET, symbol Switch:SW_Push
- added U4: XC6206P332MR, Package_TO_SOT_SMD:SOT-23, symbol kicad-keyboard-parts:XC6206PxxxMR-Regulator_Linear
- added U5: nRF52840_holyiot_18010, symbol kicad-keyboard-parts:nRF52840_holyiot_18010
- gave numbers to parts that had none: 2
Connections:
- net +5V: now also U5.22 (VBUS)
- net D+: now also U5.24 (D+)
- net D-: now also U5.23 (D-)
- net GND: now also C5.2, C6.2, C7.2, C8.2, C9.2, J3.1 (Pin_1), R11.2, SW1.2, U4.1 (GND), U5.1 (GND), U5.25 (GND), U5.37 (GND)
- net VBAT: now also R10.1
- new net: C9.1, U4.2 (VO)
- new net: C5.1, C6.1, C7.1, U4.3 (VI)
- new net: D?.2 (A), MX?.2 (ROW) (x15)
- new net: SW1.1, U5.21 (P0.18/RESET)
- new net: J3.2 (Pin_2), U5.31 (SWDCLK)
- new net: J3.3 (Pin_3), U5.32 (SWDIO)
- new net: D1.2 (A), MX1.2 (ROW)
- new net +3V3: C8.1, U5.14 (VDD_nRF)
- new net COL0: MX1.1 (COL), MX?.1 (COL), MX?.1 (COL), MX?.1 (COL)
- new net COL1: MX?.1 (COL), MX?.1 (COL), MX?.1 (COL), MX?.1 (COL), U5.36 (P0.10)
- new net COL2: MX?.1 (COL), MX?.1 (COL), MX?.1 (COL), MX?.1 (COL), U5.35 (P0.09)
- new net COL3: MX?.1 (COL), MX?.1 (COL), MX?.1 (COL), MX?.1 (COL), U5.34 (P1.06)
- new net COL4: U5.33 (P1.04)
- new net ROW0: D1.1 (K), D?.1 (K), D?.1 (K), D?.1 (K)
- new net ROW1: D?.1 (K), D?.1 (K), D?.1 (K), D?.1 (K), U5.30 (P1.02)
- new net ROW2: D?.1 (K), D?.1 (K), D?.1 (K), D?.1 (K), U5.29 (P1.01)
- new net ROW3: D?.1 (K), D?.1 (K), D?.1 (K), D?.1 (K), U5.28 (P1.03)
- new net ROW4: U5.27 (P1.00)
- new net VSENSE: R10.2, R11.1, U5.11 (P0.31)
Other:
- note added: "MCU\n"
- note added: "Switch Matrix"
- note added: "Voltage Regulator"
- note added: "\nVoltage Divider/Sensor"
- moved on the sheet: C1, C2, C3, C4, D1, D2, ESD1, F1, J1, J2, JP1, L1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

Commit message: wip
Parts:
- added RSW1, RSW2, RSW3, RSW4: EC11E, Rotary_Encoder:RotaryEncoder_Alps_EC11E-Switch_Vertical_H20mm, symbol Device:Rotary_Encoder_Switch
- added R_D1, R_D2, R_D3, R_D4: SM4007PL, random-keyboard-parts:D_SOD-123-Pretty, symbol Device:D_Small
- BD1: renamed from D1; value 1.5KExxCA -> BSD3C051V; footprint Diode_THT:D_DO-201AE_P15.24mm_Horizontal -> kicad-keyboard-parts:SOT-23_stealth
- C1, C2, C3, C4, C5, C6, C7, C8, C9: footprint (none) -> Capacitor_SMD:C_0603_1608Metric
- D1: footprint (none) -> random-keyboard-parts:D_SOD-123-Pretty
- D10, D11, D12, D13, D14, D15, D16, D2, D3, D4, D5, D6, D7, D8, D9: renamed from D?; footprint (none) -> random-keyboard-parts:D_SOD-123-Pretty
- F1: footprint (none) -> Fuse:Fuse_0603_1608Metric
- J1, J2: footprint (none) -> Connector_JST:JST_SH_SM02B-SRSS-TB_1x02-1MP_P1.00mm_Horizontal
- J3: footprint (none) -> Connector_PinHeader_2.54mm:PinHeader_1x03_P2.54mm_Vertical
- JP1: footprint (none) -> Jumper:SolderJumper-2_P1.3mm_Bridged_RoundedPad1.0x1.5mm
- L1: footprint (none) -> Inductor_SMD:L_0603_1608Metric
- LD1: renamed from D1; footprint (none) -> LED_SMD:LED_0603_1608Metric
- LD2: renamed from D2; footprint (none) -> LED_SMD:LED_0603_1608Metric
- MX1: footprint (none) -> MX_Only:MXOnly-1U-Hotswap-Antishear
- MX10, MX11, MX12, MX13, MX14, MX15, MX16, MX2, MX3, MX4, MX5, MX6, MX7, MX8, MX9: renamed from MX?; footprint (none) -> MX_Only:MXOnly-1U-Hotswap-Antishear
- R1, R10, R11, R2, R3, R4, R5, R6, R7, R8, R9: footprint (none) -> Resistor_SMD:R_0603_1608Metric
- SW1: footprint (none) -> random-keyboard-parts:SKQG-1155865
- U5: footprint (none) -> kicad-keyboard-parts:nRF52840_holyiot_18010
- USB1: footprint (none) -> Connector_USB:USB_C_Receptacle_HRO_TYPE-C-31-M-12
Connections:
- net COL4 is gone; now on net COL3: U5.33 (P1.04)
- net COL0: now also U5.36 (P0.10), RSW1.S1
- net COL1: now also U5.35 (P0.09), RSW2.S1; no longer U5.36 (P0.10)
- net COL2: now also U5.34 (P1.06), RSW3.S1; no longer U5.35 (P0.09)
- net COL3: now also RSW4.S1; no longer U5.34 (P1.06)
- net GND: now also RSW1.C, RSW2.C, RSW3.C, RSW4.C
- net ROW0: now also U5.30 (P1.02), R_D1.1 (K), R_D2.1 (K), R_D3.1 (K), R_D4.1 (K); no longer D1.1 (K), D2.1 (K), D3.1 (K), D4.1 (K)
- net ROW1: now also D1.1 (K), D2.1 (K), D3.1 (K), D4.1 (K), U5.29 (P1.01); no longer D5.1 (K), D6.1 (K), D7.1 (K), D8.1 (K), U5.30 (P1.02)
- net ROW2: now also D5.1 (K), D6.1 (K), D7.1 (K), D8.1 (K), U5.28 (P1.03); no longer D10.1 (K), D11.1 (K), D12.1 (K), D9.1 (K), U5.29 (P1.01)
- net ROW3: now also D10.1 (K), D11.1 (K), D12.1 (K), D9.1 (K), U5.27 (P1.00); no longer D13.1 (K), D14.1 (K), D15.1 (K), D16.1 (K), U5.28 (P1.03)
- net ROW4: now also D13.1 (K), D14.1 (K), D15.1 (K), D16.1 (K), U5.26 (P0.22); no longer U5.27 (P1.00)
- net VBAT: now also C5.1, C6.1, C7.1, U4.3 (VI)
- net EncA1: now reaches U5.2 (P1.11)
- net EncA1: now also RSW1.A
- net EncB1: now reaches U5.3 (P1.10)
- net EncB1: now also RSW1.B
- net EncA2: now reaches U5.4 (P1.13)
- net EncA2: now also RSW2.A
- net EncB2: now reaches U5.5 (P1.15)
- net EncB2: now also RSW2.B
- net EncA3: now reaches U5.6 (P0.03)
- net EncA3: now also RSW3.A
- net EncB3: now reaches U5.7 (P0.02)
- net EncB3: now also RSW3.B
- net EncA4: now reaches U5.8 (P0.28)
- net EncA4: now also RSW4.A
- net EncB4: now reaches U5.9 (P0.29)
- net EncB4: now also RSW4.B
- new net: RSW4.S2, R_D4.2 (A)
- new net: RSW3.S2, R_D3.2 (A)
- new net: RSW2.S2, R_D2.2 (A)
- new net: RSW1.S2, R_D1.2 (A)
- no-connect marks 7 -> 34
Other:
- note added: "ESD\n"
- note added: "Rotary Encoders Matrix\n"
- note added: "USB"
- note removed: "USB + ESD"
- moved on the sheet: BD1, C1, C2, C3, C4, C5, C6, C7, C8, C9, D1, D10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
